Commit message: #5 Change Artag Prism Now Triangular Prism

File: sdf/landmark.sdf.xacro (robot description, xacro)
@@ -3,9 +3,9 @@
   <xacro:macro name="landmark" params="id *pose">
     <xacro:property name="pole_above_ground" value="0.3"/>
-    <xacro:property name="box_width" value="0.25"/>
+    <xacro:property name="box_width" value="0.20"/>
     <xacro:property name="pole_below_ground" value="0.1"/>
     <xacro:property name="box_height" value="0.32"/>
     <xacro:property name="sheet_width" value="0.005"/> <!-- When the sheet is too thin it is not shaded properly for some reason -->
-    <xacro:property name="sheet_out" value="0.001"/>
+    <xacro:property name="sheet_out" value="0.01"/>
     <model name="landmark${id}">
       <xacro:insert_block name="pose"/>
@@ -36,9 +36,10 @@
         </collision>
         <visual name="box_visual">
-          <pose>0 0 ${pole_above_ground + box_height/2} 0 0 0</pose>
+          <pose>0 0 ${-0.15+pole_above_ground + box_height/2} 0 0 +${pi/3}</pose>
           <geometry>
-            <box>
-              <size>${box_width} ${box_width} ${box_height}</size>
-            </box>
+            <mesh>
+              <uri>/home/baran/rover_simulation_ws/src/Simulations/blender_gazebo/sdf/meshes/ERC_Sign.stl</uri> <!-- Change dictionary line-->
+              <scale>0.0013 0.0013 0.001</scale>
+            </mesh>
           </geometry>
           <material>
@@ -49,9 +50,10 @@
         </visual>
         <collision name="box_collision">
-          <pose>0 0 ${pole_above_ground + box_height/2} 0 0 0</pose>
+          <pose>0 0 ${-0.15+pole_above_ground + box_height/2} 0 0 +${pi/3}</pose>
           <geometry>
-            <box>
-              <size>${box_width} ${box_width} ${box_height}</size>
-            </box>
+            <mesh>
+              <uri>/home/baran/rover_simulation_ws/src/Simulations/blender_gazebo/sdf/meshes/ERC_Sign.stl</uri> <!-- Change dictionary line-->
+              <scale>0.0013 0.0013 0.001</scale>
+            </mesh>
           </geometry>
         </collision>
@@ -72,14 +74,14 @@
         </xacro:macro>
         <xacro:landmark_sheet name="sheet1">
-          <pose>0 ${(box_width - sheet_width)/2 + sheet_out} ${pole_above_ground + box_height/2} 0 0 0</pose>
+          <pose>0 ${(box_width - sheet_width)/2} ${pole_above_ground + box_height/2} 0 0 0</pose>
         </xacro:landmark_sheet>
-        <xacro:landmark_sheet name="sheet2">
+        <!-- <xacro:landmark_sheet name="sheet2">
           <pose>0 -${(box_width - sheet_width)/2 + sheet_out} ${pole_above_ground + box_height/2} 0 0 0</pose>
-        </xacro:landmark_sheet>
+        </xacro:landmark_sheet> -->
         <xacro:landmark_sheet name="sheet3">
-          <pose>${(box_width - sheet_width)/2 + sheet_out} 0 ${pole_above_ground + box_height/2} 0 0 ${pi/2}</pose>
+          <pose>${((box_width-0.05) - sheet_width)/2 + sheet_out} -0.06 ${pole_above_ground + box_height/2} 0 0 +${pi/3}</pose>
         </xacro:landmark_sheet>
         <xacro:landmark_sheet name="sheet4">
-          <pose>-${(box_width - sheet_width)/2 + sheet_out} 0 ${pole_above_ground + box_height/2} 0 0 ${pi/2}</pose>
+          <pose>-${((box_width-0.06) - sheet_width)/2 + sheet_out} -0.06 ${pole_above_ground + box_height/2} 0 0 -${pi/3}</pose>
         </xacro:landmark_sheet>
       </link>

File: worlds/marsyard2021.world.xacro (robot description, xacro)
@@ -25,5 +25,5 @@
       </sky>
       <shadows>true</shadows>
-      <origin_visual>false</origin_visual>
+      <origin_visual>true</origin_visual>
     </scene>
     <xacro:include filename="$(find blender_gazebo)/sdf/landmark.sdf.xacro"/>
