Commit message: #6 Gazebo Actor Added.

File: worlds/marsyard2021.world.xacro (robot description, xacro)
@@ -1,4 +1,5 @@
 <?xml version="1.0"?>
-<sdf version="1.6" xmlns:xacro="http://www.ros.org/wiki/xacro">
+<sdf version="1.6"
+  xmlns:xacro="http://www.ros.org/wiki/xacro">
   <world name="marsyard2021">
     <physics type="ode">
@@ -27,4 +28,43 @@
       <origin_visual>true</origin_visual>
     </scene>
+    <!-- <actor name="Matt Damon">
+      <link name="cosmonaut">
+        <visual name="visual">
+          <pose>0 0 0 0 0 0</pose>
+          <geometry>
+            <mesh>
+              <scale>1 1 1</scale>
+              <uri>/home/baran/rover_simulation_ws/src/Simulations/blender_gazebo/worlds/cosmonaut-dae/cosmonaut.dae</uri>
+            </mesh>
+          </geometry>
+        </visual>
+      </link>
+      <script>
+        <loop>true</loop>
+        <auto_start>true</auto_start>
+        <trajectory id="0" type="square">
+          <waypoint>
+            <time>0.0</time>
+            <pose>-1 -1 1 0 0 0</pose>
+          </waypoint>
+          <waypoint>
+            <time>1.0</time>
+            <pose>-1 1 1 0 0 0</pose>
+          </waypoint>
+          <waypoint>
+            <time>2.0</time>
+            <pose>1 1 1 0 0 0</pose>
+          </waypoint>
+          <waypoint>
+            <time>3.0</time>
+            <pose>1 -1 1 0 0 0</pose>
+          </waypoint>
+          <waypoint>
+            <time>4.0</time>
+            <pose>-1 -1 1 0 0 0</pose>
+          </waypoint>
+        </trajectory>
+      </script>
+    </actor> -->
     <xacro:include filename="$(find blender_gazebo)/sdf/landmark.sdf.xacro"/>
     <xacro:landmark id="1">
